Commit message: Added Camera to the Bot

File: bd1_bot_description/urdf/bd1_bot.xacro (robot description, xacro)
@@ -26,7 +26,7 @@
 <link name="left_top_leg_1">
   <inertial>
-    <origin xyz="0.008147102971613814 0.029774274347874285 -0.02977410630349306" rpy="0 0 0"/>
+    <origin xyz="0.008147102971613904 0.03956774889582286 -0.014401430555830014" rpy="0 0 0"/>
     <mass value="0.15317289375951978"/>
-    <inertia ixx="0.00031" iyy="0.000159" izz="0.000159" ixy="-6e-06" iyz="0.000114" ixz="6e-06"/>
+    <inertia ixx="0.00031" iyy="7.2e-05" izz="0.000247" ixy="-8e-06" iyz="7.3e-05" ixz="3e-06"/>
   </inertial>
   <visual>
@@ -46,7 +46,7 @@
 <link name="right_top_leg_1">
   <inertial>
-    <origin xyz="-0.008146173310383559 0.029774274348084395 -0.029774106303283948" rpy="0 0 0"/>
+    <origin xyz="-0.008146173310383482 0.03956774889592504 -0.014401430555552125" rpy="0 0 0"/>
     <mass value="0.15317289375951978"/>
-    <inertia ixx="0.00031" iyy="0.000159" izz="0.000159" ixy="6e-06" iyz="0.000114" ixz="-6e-06"/>
+    <inertia ixx="0.00031" iyy="7.2e-05" izz="0.000247" ixy="8e-06" iyz="7.3e-05" ixz="-3e-06"/>
   </inertial>
   <visual>
@@ -66,10 +66,10 @@
 <link name="left_top_leg_part_1">
   <inertial>
-    <origin xyz="0.003017147690063067 -0.005386994713906336 0.0053871627584965165" rpy="0 0 0"/>
+    <origin xyz="0.0030171476900631364 -0.00715861722472852 0.002605715273466813" rpy="0 0 0"/>
     <mass value="0.0046248042940224615"/>
-    <inertia ixx="2e-06" iyy="1e-06" izz="1e-06" ixy="0.0" iyz="1e-06" ixz="-0.0"/>
-  </inertial>
-  <visual>
-    <origin xyz="-0.057454 -0.039829 -0.169306" rpy="0 0 0"/>
+    <inertia ixx="2e-06" iyy="0.0" izz="2e-06" ixy="0.0" iyz="1e-06" ixz="-0.0"/>
+  </inertial>
+  <visual>
+    <origin xyz="-0.057454 -0.049902 -0.185118" rpy="0 0 0"/>
     <geometry>
       <mesh filename="file://$(find bd1_bot_description)/meshes/left_top_leg_part_1.stl" scale="0.001 0.001 0.001"/>
@@ -78,5 +78,5 @@
   </visual>
   <collision>
-    <origin xyz="-0.057454 -0.039829 -0.169306" rpy="0 0 0"/>
+    <origin xyz="-0.057454 -0.049902 -0.185118" rpy="0 0 0"/>
     <geometry>
       <mesh filename="file://$(find bd1_bot_description)/meshes/left_top_leg_part_1.stl" scale="0.001 0.001 0.001"/>
@@ -86,10 +86,10 @@
 <link name="right_top_leg_part_1">
   <inertial>
-    <origin xyz="-0.0030162180288329024 -0.005386994713905212 0.005387162758496544" rpy="0 0 0"/>
+    <origin xyz="-0.00301621802883284 -0.0071586172247272845 0.0026057152734667854" rpy="0 0 0"/>
     <mass value="0.0046248042940224615"/>
-    <inertia ixx="2e-06" iyy="1e-06" izz="1e-06" ixy="-0.0" iyz="1e-06" ixz="0.0"/>
-  </inertial>
-  <visual>
-    <origin xyz="0.058046 -0.039829 -0.169306" rpy="0 0 0"/>
+    <inertia ixx="2e-06" iyy="0.0" izz="2e-06" ixy="-0.0" iyz="1e-06" ixz="0.0"/>
+  </inertial>
+  <visual>
+    <origin xyz="0.058046 -0.049902 -0.185118" rpy="0 0 0"/>
     <geometry>
       <mesh filename="file://$(find bd1_bot_description)/meshes/right_top_leg_part_1.stl" scale="0.001 0.001 0.001"/>
@@ -98,5 +98,5 @@
   </visual>
   <collision>
-    <origin xyz="0.058046 -0.039829 -0.169306" rpy="0 0 0"/>
+    <origin xyz="0.058046 -0.049902 -0.185118" rpy="0 0 0"/>
     <geometry>
       <mesh filename="file://$(find bd1_bot_description)/meshes/right_top_leg_part_1.stl" scale="0.001 0.001 0.001"/>
@@ -106,10 +106,10 @@
 <link name="left_bottom_leg_1">
   <inertial>
-    <origin xyz="-0.004999535169384957 -0.040779246943576826 -0.03875617837865104" rpy="0 0 0"/>
+    <origin xyz="-0.004999535169384679 -0.031830123018515816 -0.046387815622354014" rpy="0 0 0"/>
     <mass value="0.08714904531938553"/>
-    <inertia ixx="0.0002" iyy="9.7e-05" izz="0.000105" ixy="-0.0" iyz="-8.2e-05" ixz="-0.0"/>
-  </inertial>
-  <visual>
-    <origin xyz="-0.043454 -0.078147 -0.130988" rpy="0 0 0"/>
+    <inertia ixx="0.0002" iyy="0.00013" izz="7.1e-05" ixy="-0.0" iyz="-7.6e-05" ixz="-0.0"/>
+  </inertial>
+  <visual>
+    <origin xyz="-0.043454 -0.100824 -0.166584" rpy="0 0 0"/>
     <geometry>
       <mesh filename="file://$(find bd1_bot_description)/meshes/left_bottom_leg_1.stl" scale="0.001 0.001 0.001"/>
@@ -118,5 +118,5 @@
   </visual>
   <collision>
-    <origin xyz="-0.043454 -0.078147 -0.130988" rpy="0 0 0"/>
+    <origin xyz="-0.043454 -0.100824 -0.166584" rpy="0 0 0"/>
     <geometry>
       <mesh filename="file://$(find bd1_bot_description)/meshes/left_bottom_leg_1.stl" scale="0.001 0.001 0.001"/>
@@ -126,10 +126,10 @@
 <link name="right_bottom_leg_1">
   <inertial>
-    <origin xyz="0.004000464830615183 -0.04077924694357608 -0.03875617837865103" rpy="0 0 0"/>
+    <origin xyz="0.0040004648306154605 -0.031830123018515136 -0.04638781562235404" rpy="0 0 0"/>
     <mass value="0.08714904531938553"/>
-    <inertia ixx="0.0002" iyy="9.7e-05" izz="0.000105" ixy="-0.0" iyz="-8.2e-05" ixz="-0.0"/>
-  </inertial>
-  <visual>
-    <origin xyz="0.044046 -0.078147 -0.130988" rpy="0 0 0"/>
+    <inertia ixx="0.0002" iyy="0.00013" izz="7.1e-05" ixy="-0.0" iyz="-7.6e-05" ixz="-0.0"/>
+  </inertial>
+  <visual>
+    <origin xyz="0.044046 -0.100824 -0.166584" rpy="0 0 0"/>
     <geometry>
       <mesh filename="file://$(find bd1_bot_description)/meshes/right_bottom_leg_1.stl" scale="0.001 0.001 0.001"/>
@@ -138,5 +138,5 @@
   </visual>
   <collision>
-    <origin xyz="0.044046 -0.078147 -0.130988" rpy="0 0 0"/>
+    <origin xyz="0.044046 -0.100824 -0.166584" rpy="0 0 0"/>
     <geometry>
       <mesh filename="file://$(find bd1_bot_description)/meshes/right_bottom_leg_1.stl" scale="0.001 0.001 0.001"/>
@@ -146,10 +146,10 @@
 <link name="right_bottom_leg_part1_1">
   <inertial>
-    <origin xyz="-0.002888264879339089 0.040001717309939545 0.04000169899847817" rpy="0 0 0"/>
+    <origin xyz="-0.0028882648793387977 0.03081062641368465 0.047444536625710965" rpy="0 0 0"/>
     <mass value="0.01039775817481047"/>
-    <inertia ixx="1.3e-05" iyy="6e-06" izz="6e-06" ixy="0.0" iyz="-6e-06" ixz="0.0"/>
-  </inertial>
-  <visual>
-    <origin xyz="0.044046 0.00317 -0.049671" rpy="0 0 0"/>
+    <inertia ixx="1.3e-05" iyy="9e-06" izz="4e-06" ixy="0.0" iyz="-5e-06" ixz="0.0"/>
+  </inertial>
+  <visual>
+    <origin xyz="0.044046 -0.038191 -0.070137" rpy="0 0 0"/>
     <geometry>
       <mesh filename="file://$(find bd1_bot_description)/meshes/right_bottom_leg_part1_1.stl" scale="0.001 0.001 0.001"/>
@@ -158,5 +158,5 @@
   </visual>
   <collision>
-    <origin xyz="0.044046 0.00317 -0.049671" rpy="0 0 0"/>
+    <origin xyz="0.044046 -0.038191 -0.070137" rpy="0 0 0"/>
     <geometry>
       <mesh filename="file://$(find bd1_bot_description)/meshes/right_bottom_leg_part1_1.stl" scale="0.001 0.001 0.001"/>
@@ -166,10 +166,10 @@
 <link name="right_bottom_leg_part2_1">
   <inertial>
-    <origin xyz="0.0028891945405694133 0.04000171730993943 0.040001698998478157" rpy="0 0 0"/>
+    <origin xyz="0.002889194540569691 0.030810626413684525 0.04744453662571095" rpy="0 0 0"/>
     <mass value="0.01039775817481047"/>
-    <inertia ixx="1.3e-05" iyy="6e-06" izz="6e-06" ixy="-0.0" iyz="-6e-06" ixz="-0.0"/>
-  </inertial>
-  <visual>
-    <origin xyz="0.036046 0.00317 -0.049671" rpy="0 0 0"/>
+    <inertia ixx="1.3e-05" iyy="9e-06" izz="4e-06" ixy="-0.0" iyz="-5e-06" ixz="-0.0"/>
+  </inertial>
+  <visual>
+    <origin xyz="0.036046 -0.038191 -0.070137" rpy="0 0 0"/>
     <geometry>
       <mesh filename="file://$(find bd1_bot_description)/meshes/right_bottom_leg_part2_1.stl" scale="0.001 0.001 0.001"/>
@@ -178,5 +178,5 @@
   </visual>
   <collision>
-    <origin xyz="0.036046 0.00317 -0.049671" rpy="0 0 0"/>
+    <origin xyz="0.036046 -0.038191 -0.070137" rpy="0 0 0"/>
     <geometry>
       <mesh filename="file://$(find bd1_bot_description)/meshes/right_bottom_leg_part2_1.stl" scale="0.001 0.001 0.001"/>
@@ -186,10 +186,10 @@
 <link name="left_bottom_leg_part1_1">
   <inertial>
-    <origin xyz="0.0028891945405692815 0.040001717309938664 0.04000169899847814" rpy="0 0 0"/>
+    <origin xyz="0.002889194540569559 0.030810626413683845 0.04744453662571098" rpy="0 0 0"/>
     <mass value="0.01039775817481047"/>
-    <inertia ixx="1.3e-05" iyy="6e-06" izz="6e-06" ixy="-0.0" iyz="-6e-06" ixz="-0.0"/>
-  </inertial>
-  <visual>
-    <origin xyz="-0.042454 0.00317 -0.049671" rpy="0 0 0"/>
+    <inertia ixx="1.3e-05" iyy="9e-06" izz="4e-06" ixy="-0.0" iyz="-5e-06" ixz="-0.0"/>
+  </inertial>
+  <visual>
+    <origin xyz="-0.042454 -0.038191 -0.070137" rpy="0 0 0"/>
     <geometry>
       <mesh filename="file://$(find bd1_bot_description)/meshes/left_bottom_leg_part1_1.stl" scale="0.001 0.001 0.001"/>
@@ -198,5 +198,5 @@
   </visual>
   <collision>
-    <origin xyz="-0.042454 0.00317 -0.049671" rpy="0 0 0"/>
+    <origin xyz="-0.042454 -0.038191 -0.070137" rpy="0 0 0"/>
     <geometry>
       <mesh filename="file://$(find bd1_bot_description)/meshes/left_bottom_leg_part1_1.stl" scale="0.001 0.001 0.001"/>
@@ -206,10 +206,10 @@
 <link name="left_bottom_leg_part2_1">
   <inertial>
-    <origin xyz="-0.002888264879339214 0.04000171730993878 0.04000169899847814" rpy="0 0 0"/>
+    <origin xyz="-0.0028882648793389296 0.030810626413683984 0.047444536625710965" rpy="0 0 0"/>
     <mass value="0.01039775817481047"/>
-    <inertia ixx="1.3e-05" iyy="6e-06" izz="6e-06" ixy="0.0" iyz="-6e-06" ixz="0.0"/>
-  </inertial>
-  <visual>
-    <origin xyz="-0.034454 0.00317 -0.049671" rpy="0 0 0"/>
+    <inertia ixx="1.3e-05" iyy="9e-06" izz="4e-06" ixy="0.0" iyz="-5e-06" ixz="0.0"/>
+  </inertial>
+  <visual>
+    <origin xyz="-0.034454 -0.038191 -0.070137" rpy="0 0 0"/>
     <geometry>
       <mesh filename="file://$(find bd1_bot_description)/meshes/left_bottom_leg_part2_1.stl" scale="0.001 0.001 0.001"/>
@@ -218,5 +218,5 @@
   </visual>
   <collision>
-    <origin xyz="-0.034454 0.00317 -0.049671" rpy="0 0 0"/>
+    <origin xyz="-0.034454 -0.038191 -0.070137" rpy="0 0 0"/>
     <geometry>
       <mesh filename="file://$(find bd1_bot_description)/meshes/left_bottom_leg_part2_1.stl" scale="0.001 0.001 0.001"/>
@@ -226,10 +226,10 @@
 <link name="left_motor_1">
   <inertial>
-    <origin xyz="0.015112405129122049 2.1162377481301342e-07 1.9331231316394026e-07" rpy="0 0 0"/>
+    <origin xyz="0.015112405129122444 1.3798701027981086e-07 -1.5177490494955315e-07" rpy="0 0 0"/>
     <mass value="0.1704942333103181"/>
     <inertia ixx="1.9e-05" iyy="2.3e-05" izz="2.3e-05" ixy="-0.0" iyz="0.0" ixz="0.0"/>
   </inertial>
   <visual>
-    <origin xyz="-0.029454 0.013777 -0.039064" rpy="0 0 0"/>
+    <origin xyz="-0.029454 -0.030021 -0.057557" rpy="0 0 0"/>
     <geometry>
       <mesh filename="file://$(find bd1_bot_description)/meshes/left_motor_1.stl" scale="0.001 0.001 0.001"/>
@@ -238,5 +238,5 @@
   </visual>
   <collision>
-    <origin xyz="-0.029454 0.013777 -0.039064" rpy="0 0 0"/>
+    <origin xyz="-0.029454 -0.030021 -0.057557" rpy="0 0 0"/>
     <geometry>
       <mesh filename="file://$(find bd1_bot_description)/meshes/left_motor_1.stl" scale="0.001 0.001 0.001"/>
@@ -246,10 +246,10 @@
 <link name="right_motor_1">
   <inertial>
-    <origin xyz="-0.015111475467892755 2.116237745822952e-07 1.9331231430885776e-07" rpy="0 0 0"/>
+    <origin xyz="-0.015111475467892387 1.3798700971776046e-07 -1.5177490413770256e-07" rpy="0 0 0"/>
     <mass value="0.1704942333103181"/>
     <inertia ixx="1.9e-05" iyy="2.3e-05" izz="2.3e-05" ixy="-0.0" iyz="0.0" ixz="0.0"/>
   </inertial>
   <visual>
-    <origin xyz="0.031046 0.013777 -0.039064" rpy="0 0 0"/>
+    <origin xyz="0.031046 -0.030021 -0.057557" rpy="0 0 0"/>
     <geometry>
       <mesh filename="file://$(find bd1_bot_description)/meshes/right_motor_1.stl" scale="0.001 0.001 0.001"/>
@@ -258,5 +258,5 @@
   </visual>
   <collision>
-    <origin xyz="0.031046 0.013777 -0.039064" rpy="0 0 0"/>
+    <origin xyz="0.031046 -0.030021 -0.057557" rpy="0 0 0"/>
     <geometry>
       <mesh filename="file://$(find bd1_bot_description)/meshes/right_motor_1.stl" scale="0.001 0.001 0.001"/>
@@ -266,10 +266,10 @@
 <link name="left_wheel_1">
   <inertial>
-    <origin xyz="-0.004999534893302154 2.0516767676968806e-07 1.8739455825977913e-07" rpy="0 0 0"/>
+    <origin xyz="-0.004999534893301766 1.329023638918514e-07 -1.5890564092346793e-07" rpy="0 0 0"/>
     <mass value="0.04003018480536562"/>
-    <inertia ixx="2.8e-05" iyy="1.5e-05" izz="1.5e-05" ixy="-0.0" iyz="0.0" ixz="-0.0"/>
-  </inertial>
-  <visual>
-    <origin xyz="-0.074454 0.013777 -0.039064" rpy="0 0 0"/>
+    <inertia ixx="2.8e-05" iyy="1.5e-05" izz="1.5e-05" ixy="-0.0" iyz="-0.0" ixz="-0.0"/>
+  </inertial>
+  <visual>
+    <origin xyz="-0.074454 -0.030021 -0.057557" rpy="0 0 0"/>
     <geometry>
       <mesh filename="file://$(find bd1_bot_description)/meshes/left_wheel_1.stl" scale="0.001 0.001 0.001"/>
@@ -278,5 +278,5 @@
   </visual>
   <collision>
-    <origin xyz="-0.074454 0.013777 -0.039064" rpy="0 0 0"/>
+    <origin xyz="-0.074454 -0.030021 -0.057557" rpy="0 0 0"/>
     <geometry>
       <mesh filename="file://$(find bd1_bot_description)/meshes/left_wheel_1.stl" scale="0.001 0.001 0.001"/>
@@ -286,10 +286,10 @@
 <link name="right_wheel_1">
   <inertial>
-    <origin xyz="0.0050004645545314585 2.057060199019134e-07 1.8685621649278117e-07" rpy="0 0 0"/>
+    <origin xyz="0.005000464554531833 1.3354087039299523e-07 -1.593202911612246e-07" rpy="0 0 0"/>
     <mass value="0.04003018480536562"/>
     <inertia ixx="2.8e-05" iyy="1.5e-05" izz="1.5e-05" ixy="0.0" iyz="0.0" ixz="0.0"/>
   </inertial>
   <visual>
-    <origin xyz="0.076046 0.013777 -0.039064" rpy="0 0 0"/>
+    <origin xyz="0.076046 -0.030021 -0.057557" rpy="0 0 0"/>
     <geometry>
       <mesh filename="file://$(find bd1_bot_description)/meshes/right_wheel_1.stl" scale="0.001 0.001 0.001"/>
@@ -298,5 +298,5 @@
   </visual>
   <collision>
-    <origin xyz="0.076046 0.013777 -0.039064" rpy="0 0 0"/>
+    <origin xyz="0.076046 -0.030021 -0.057557" rpy="0 0 0"/>
     <geometry>
       <mesh filename="file://$(find bd1_bot_description)/meshes/right_wheel_1.stl" scale="0.001 0.001 0.001"/>
@@ -306,10 +306,10 @@
 <link name="left_tyre_1">
   <inertial>
-    <origin xyz="0.010019051332744715 2.1211038524204806e-07 1.9375316993169855e-07" rpy="0 0 0"/>
-    <mass value="0.024103944434888665"/>
+    <origin xyz="0.010019081554393537 1.3838490093773248e-07 -1.512219713339924e-07" rpy="0 0 0"/>
+    <mass value="0.024104122361266803"/>
     <inertia ixx="2.9e-05" iyy="1.6e-05" izz="1.6e-05" ixy="-0.0" iyz="-0.0" ixz="-0.0"/>
   </inertial>
   <visual>
-    <origin xyz="-0.059454 0.013777 -0.039064" rpy="0 0 0"/>
+    <origin xyz="-0.059454 -0.030021 -0.057557" rpy="0 0 0"/>
     <geometry>
       <mesh filename="file://$(find bd1_bot_description)/meshes/left_tyre_1.stl" scale="0.001 0.001 0.001"/>
@@ -318,5 +318,5 @@
   </visual>
   <collision>
-    <origin xyz="-0.059454 0.013777 -0.039064" rpy="0 0 0"/>
+    <origin xyz="-0.059454 -0.030021 -0.057557" rpy="0 0 0"/>
     <geometry>
       <mesh filename="file://$(find bd1_bot_description)/meshes/left_tyre_1.stl" scale="0.001 0.001 0.001"/>
@@ -326,10 +326,10 @@
 <link name="right_tyre_1">
   <inertial>
-    <origin xyz="-0.010018121671515418 2.1118291914160037e-07 1.9282570255102494e-07" rpy="0 0 0"/>
-    <mass value="0.024103944434888665"/>
+    <origin xyz="-0.010018151893163477 1.3764371806571085e-07 -1.5236329475865062e-07" rpy="0 0 0"/>
+    <mass value="0.024104122361266803"/>
     <inertia ixx="2.9e-05" iyy="1.6e-05" izz="1.6e-05" ixy="-0.0" iyz="-0.0" ixz="-0.0"/>
   </inertial>
   <visual>
-    <origin xyz="0.061046 0.013777 -0.039064" rpy="0 0 0"/>
+    <origin xyz="0.061046 -0.030021 -0.057557" rpy="0 0 0"/>
     <geometry>
       <mesh filename="file://$(find bd1_bot_description)/meshes/right_tyre_1.stl" scale="0.001 0.001 0.001"/>
@@ -338,5 +338,5 @@
   </visual>
   <collision>
-    <origin xyz="0.061046 0.013777 -0.039064" rpy="0 0 0"/>
+    <origin xyz="0.061046 -0.030021 -0.057557" rpy="0 0 0"/>
     <geometry>
       <mesh filename="file://$(find bd1_bot_description)/meshes/right_tyre_1.stl" scale="0.001 0.001 0.001"/>
@@ -366,6 +366,6 @@
 <link name="head_1">
   <inertial>
-    <origin xyz="0.005426321856642208 -0.021648994769970266 0.009088552143427908" rpy="0 0 0"/>
-    <mass value="1.5697512261294357"/>
+    <origin xyz="0.005426334184364864 -0.021649063420818744 0.009088570503094973" rpy="0 0 0"/>
+    <mass value="1.569749070523499"/>
     <inertia ixx="0.004122" iyy="0.003236" izz="0.006741" ixy="-1e-06" iyz="6.5e-05" ixz="-3e-06"/>
   </inertial>
@@ -446,6 +446,6 @@
 <link name="head_display_1">
   <inertial>
-    <origin xyz="0.00035190281604508336 0.003044468925605781 -0.0025415429702123626" rpy="0 0 0"/>
-    <mass value="0.008893910243592446"/>
+    <origin xyz="0.00035190281604519005 0.003044468925605781 -0.002541542970212418" rpy="0 0 0"/>
+    <mass value="0.008893910243592436"/>
     <inertia ixx="1e-06" iyy="1.8e-05" izz="1.7e-05" ixy="0.0" iyz="0.0" ixz="-0.0"/>
   </inertial>
@@ -583,4 +583,44 @@
     </geometry>
   </collision>
+</link>
+<link name="ov_camera_1">
+  <inertial>
+    <origin xyz="-0.0006538876382471456 -0.005661900815445056 0.0017258208227936833" rpy="0 0 0"/>
+    <mass value="0.006421856007710609"/>
+    <inertia ixx="1e-06" iyy="1e-06" izz="1e-06" ixy="0.0" iyz="-0.0" ixz="0.0"/>
+  </inertial>
+  <visual>
+    <origin xyz="0.000296 0.061142 -0.201481" rpy="0 0 0"/>
+    <geometry>
+      <mesh filename="file://$(find bd1_bot_description)/meshes/ov_camera_1.stl" scale="0.001 0.001 0.001"/>
+    </geometry>
+    <material name="silver"/>
+  </visual>
+  <collision>
+    <origin xyz="0.000296 0.061142 -0.201481" rpy="0 0 0"/>
+    <geometry>
+      <mesh filename="file://$(find bd1_bot_description)/meshes/ov_camera_1.stl" scale="0.001 0.001 0.001"/>
+    </geometry>
+  </collision>
+</link>
+<link name="fake_camera_1">
+  <inertial>
+    <origin xyz="-0.0006538876382471456 -0.005661900815445056 0.0017258208227936833" rpy="0 0 0"/>
+    <mass value="0.006421856007710609"/>
+    <inertia ixx="1e-06" iyy="1e-06" izz="1e-06" ixy="0.0" iyz="-0.0" ixz="0.0"/>
+  </inertial>
+  <!-- <visual>
+    <origin xyz="0.000296 0.061142 -0.201481" rpy="0 0 0"/>
+    <geometry>
+      <mesh filename="file://$(find bd1_bot_description)/meshes/ov_camera_1.stl" scale="0.001 0.001 0.001"/>
+    </geometry>
+    <material name="silver"/>
+  </visual>
+  <collision>
+    <origin xyz="0.000296 0.061142 -0.201481" rpy="0 0 0"/>
+    <geometry>
+      <mesh filename="file://$(find bd1_bot_description)/meshes/ov_camera_1.stl" scale="0.001 0.001 0.001"/>
+    </geometry>
+  </collision> -->
 </link>
 <joint name="left_head_leg_fix" type="fixed">
@@ -595,50 +635,50 @@
 </joint>
 <joint name="left_head_part_fix" type="fixed">
-  <origin xyz="0.014 0.030625 -0.030625" rpy="0 0 0"/>
+  <origin xyz="0.014 0.040698 -0.014813" rpy="0 0 0"/>
   <parent link="left_top_leg_1"/>
   <child link="left_top_leg_part_1"/>
 </joint>
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