Commit message: Updated design Files

File: bd1_bot_description/urdf/bd1_bot.xacro (robot description, xacro)
@@ -6,7 +6,7 @@
 <link name="base_link">
   <inertial>
-    <origin xyz="-0.00032734350998174234 -0.00267829787408143 0.20026482146590865" rpy="0 0 0"/>
-    <mass value="0.8946153977936162"/>
-    <inertia ixx="0.001664" iyy="0.000982" izz="0.001596" ixy="0.0" iyz="1.2e-05" ixz="-1e-06"/>
+    <origin xyz="-0.00032734350998203383 -0.03347164637300757 0.1802949431054025" rpy="0 0 0"/>
+    <mass value="0.6871683490298791"/>
+    <inertia ixx="0.001278" iyy="0.000754" izz="0.001226" ixy="0.0" iyz="9e-06" ixz="-0.0"/>
   </inertial>
   <visual>
@@ -26,10 +26,10 @@
 <link name="left_top_leg_1">
   <inertial>
-    <origin xyz="0.008147102971613904 0.03956774889582286 -0.014401430555830014" rpy="0 0 0"/>
-    <mass value="0.15317289375951978"/>
-    <inertia ixx="0.00031" iyy="7.2e-05" izz="0.000247" ixy="-8e-06" iyz="7.3e-05" ixz="3e-06"/>
-  </inertial>
-  <visual>
-    <origin xyz="-0.043454 -0.009204 -0.199931" rpy="0 0 0"/>
+    <origin xyz="0.008147102971613591 0.039567400396896726 -0.014401308916336203" rpy="0 0 0"/>
+    <mass value="0.11765454158339926"/>
+    <inertia ixx="0.000238" iyy="5.5e-05" izz="0.000189" ixy="-6e-06" iyz="5.6e-05" ixz="2e-06"/>
+  </inertial>
+  <visual>
+    <origin xyz="-0.043454 0.021589 -0.179961" rpy="0 0 0"/>
     <geometry>
       <mesh filename="file://$(find bd1_bot_description)/meshes/left_top_leg_1.stl" scale="0.001 0.001 0.001"/>
@@ -38,5 +38,5 @@
   </visual>
   <collision>
-    <origin xyz="-0.043454 -0.009204 -0.199931" rpy="0 0 0"/>
+    <origin xyz="-0.043454 0.021589 -0.179961" rpy="0 0 0"/>
     <geometry>
       <mesh filename="file://$(find bd1_bot_description)/meshes/left_top_leg_1.stl" scale="0.001 0.001 0.001"/>
@@ -46,10 +46,10 @@
 <link name="right_top_leg_1">
   <inertial>
-    <origin xyz="-0.008146173310383482 0.03956774889592504 -0.014401430555552125" rpy="0 0 0"/>
-    <mass value="0.15317289375951978"/>
-    <inertia ixx="0.00031" iyy="7.2e-05" izz="0.000247" ixy="8e-06" iyz="7.3e-05" ixz="-3e-06"/>
-  </inertial>
-  <visual>
-    <origin xyz="0.044046 -0.009204 -0.199931" rpy="0 0 0"/>
+    <origin xyz="-0.008146173310383774 0.03956740039699889 -0.014401308916058286" rpy="0 0 0"/>
+    <mass value="0.11765454158339926"/>
+    <inertia ixx="0.000238" iyy="5.5e-05" izz="0.000189" ixy="6e-06" iyz="5.6e-05" ixz="-2e-06"/>
+  </inertial>
+  <visual>
+    <origin xyz="0.044046 0.021589 -0.179961" rpy="0 0 0"/>
     <geometry>
       <mesh filename="file://$(find bd1_bot_description)/meshes/right_top_leg_1.stl" scale="0.001 0.001 0.001"/>
@@ -58,5 +58,5 @@
   </visual>
   <collision>
-    <origin xyz="0.044046 -0.009204 -0.199931" rpy="0 0 0"/>
+    <origin xyz="0.044046 0.021589 -0.179961" rpy="0 0 0"/>
     <geometry>
       <mesh filename="file://$(find bd1_bot_description)/meshes/right_top_leg_1.stl" scale="0.001 0.001 0.001"/>
@@ -66,10 +66,10 @@
 <link name="left_top_leg_part_1">
   <inertial>
-    <origin xyz="0.0030171476900631364 -0.00715861722472852 0.002605715273466813" rpy="0 0 0"/>
-    <mass value="0.0046248042940224615"/>
-    <inertia ixx="2e-06" iyy="0.0" izz="2e-06" ixy="0.0" iyz="1e-06" ixz="-0.0"/>
-  </inertial>
-  <visual>
-    <origin xyz="-0.057454 -0.049902 -0.185118" rpy="0 0 0"/>
+    <origin xyz="0.003017147690062824 -0.007158965723654645 0.002605836912960652" rpy="0 0 0"/>
+    <mass value="0.00355238590700276"/>
+    <inertia ixx="1e-06" iyy="0.0" izz="1e-06" ixy="0.0" iyz="0.0" ixz="-0.0"/>
+  </inertial>
+  <visual>
+    <origin xyz="-0.057454 -0.019109 -0.165148" rpy="0 0 0"/>
     <geometry>
       <mesh filename="file://$(find bd1_bot_description)/meshes/left_top_leg_part_1.stl" scale="0.001 0.001 0.001"/>
@@ -78,5 +78,5 @@
   </visual>
   <collision>
-    <origin xyz="-0.057454 -0.049902 -0.185118" rpy="0 0 0"/>
+    <origin xyz="-0.057454 -0.019109 -0.165148" rpy="0 0 0"/>
     <geometry>
       <mesh filename="file://$(find bd1_bot_description)/meshes/left_top_leg_part_1.stl" scale="0.001 0.001 0.001"/>
@@ -86,10 +86,10 @@
 <link name="right_top_leg_part_1">
   <inertial>
-    <origin xyz="-0.00301621802883284 -0.0071586172247272845 0.0026057152734667854" rpy="0 0 0"/>
-    <mass value="0.0046248042940224615"/>
-    <inertia ixx="2e-06" iyy="0.0" izz="2e-06" ixy="-0.0" iyz="1e-06" ixz="0.0"/>
-  </inertial>
-  <visual>
-    <origin xyz="0.058046 -0.049902 -0.185118" rpy="0 0 0"/>
+    <origin xyz="-0.0030162180288331314 -0.007158965723653446 0.002605836912960652" rpy="0 0 0"/>
+    <mass value="0.00355238590700276"/>
+    <inertia ixx="1e-06" iyy="0.0" izz="1e-06" ixy="-0.0" iyz="0.0" ixz="0.0"/>
+  </inertial>
+  <visual>
+    <origin xyz="0.058046 -0.019109 -0.165148" rpy="0 0 0"/>
     <geometry>
       <mesh filename="file://$(find bd1_bot_description)/meshes/right_top_leg_part_1.stl" scale="0.001 0.001 0.001"/>
@@ -98,5 +98,5 @@
   </visual>
   <collision>
-    <origin xyz="0.058046 -0.049902 -0.185118" rpy="0 0 0"/>
+    <origin xyz="0.058046 -0.019109 -0.165148" rpy="0 0 0"/>
     <geometry>
       <mesh filename="file://$(find bd1_bot_description)/meshes/right_top_leg_part_1.stl" scale="0.001 0.001 0.001"/>
@@ -106,10 +106,10 @@
 <link name="left_bottom_leg_1">
   <inertial>
-    <origin xyz="-0.004999535169384679 -0.031830123018515816 -0.046387815622354014" rpy="0 0 0"/>
-    <mass value="0.08714904531938553"/>
-    <inertia ixx="0.0002" iyy="0.00013" izz="7.1e-05" ixy="-0.0" iyz="-7.6e-05" ixz="-0.0"/>
-  </inertial>
-  <visual>
-    <origin xyz="-0.043454 -0.100824 -0.166584" rpy="0 0 0"/>
+    <origin xyz="-0.004999535169384971 -0.03183047151744199 -0.046387693982860134" rpy="0 0 0"/>
+    <mass value="0.06694057104242657"/>
+    <inertia ixx="0.000154" iyy="0.0001" izz="5.5e-05" ixy="-0.0" iyz="-5.9e-05" ixz="-0.0"/>
+  </inertial>
+  <visual>
+    <origin xyz="-0.043454 -0.070031 -0.146614" rpy="0 0 0"/>
     <geometry>
       <mesh filename="file://$(find bd1_bot_description)/meshes/left_bottom_leg_1.stl" scale="0.001 0.001 0.001"/>
@@ -118,5 +118,5 @@
   </visual>
   <collision>
-    <origin xyz="-0.043454 -0.100824 -0.166584" rpy="0 0 0"/>
+    <origin xyz="-0.043454 -0.070031 -0.146614" rpy="0 0 0"/>
     <geometry>
       <mesh filename="file://$(find bd1_bot_description)/meshes/left_bottom_leg_1.stl" scale="0.001 0.001 0.001"/>
@@ -126,10 +126,10 @@
 <link name="right_bottom_leg_1">
   <inertial>
-    <origin xyz="0.0040004648306154605 -0.031830123018515136 -0.04638781562235404" rpy="0 0 0"/>
-    <mass value="0.08714904531938553"/>
-    <inertia ixx="0.0002" iyy="0.00013" izz="7.1e-05" ixy="-0.0" iyz="-7.6e-05" ixz="-0.0"/>
-  </inertial>
-  <visual>
-    <origin xyz="0.044046 -0.100824 -0.166584" rpy="0 0 0"/>
+    <origin xyz="0.004000464830615148 -0.03183047151744129 -0.04638769398286016" rpy="0 0 0"/>
+    <mass value="0.06694057104242657"/>
+    <inertia ixx="0.000154" iyy="0.0001" izz="5.5e-05" ixy="-0.0" iyz="-5.9e-05" ixz="-0.0"/>
+  </inertial>
+  <visual>
+    <origin xyz="0.044046 -0.070031 -0.146614" rpy="0 0 0"/>
     <geometry>
       <mesh filename="file://$(find bd1_bot_description)/meshes/right_bottom_leg_1.stl" scale="0.001 0.001 0.001"/>
@@ -138,5 +138,5 @@
   </visual>
   <collision>
-    <origin xyz="0.044046 -0.100824 -0.166584" rpy="0 0 0"/>
+    <origin xyz="0.044046 -0.070031 -0.146614" rpy="0 0 0"/>
     <geometry>
       <mesh filename="file://$(find bd1_bot_description)/meshes/right_bottom_leg_1.stl" scale="0.001 0.001 0.001"/>
@@ -146,10 +146,10 @@
 <link name="right_bottom_leg_part1_1">
   <inertial>
-    <origin xyz="-0.0028882648793387977 0.03081062641368465 0.047444536625710965" rpy="0 0 0"/>
-    <mass value="0.01039775817481047"/>
-    <inertia ixx="1.3e-05" iyy="9e-06" izz="4e-06" ixy="0.0" iyz="-5e-06" ixz="0.0"/>
-  </inertial>
-  <visual>
-    <origin xyz="0.044046 -0.038191 -0.070137" rpy="0 0 0"/>
+    <origin xyz="-0.002888264879339103 0.030811277914758503 0.04744465826520482" rpy="0 0 0"/>
+    <mass value="0.00798668381543413"/>
+    <inertia ixx="1e-05" iyy="7e-06" izz="3e-06" ixy="0.0" iyz="-4e-06" ixz="0.0"/>
+  </inertial>
+  <visual>
+    <origin xyz="0.044046 -0.007397 -0.050167" rpy="0 0 0"/>
     <geometry>
       <mesh filename="file://$(find bd1_bot_description)/meshes/right_bottom_leg_part1_1.stl" scale="0.001 0.001 0.001"/>
@@ -158,5 +158,5 @@
   </visual>
   <collision>
-    <origin xyz="0.044046 -0.038191 -0.070137" rpy="0 0 0"/>
+    <origin xyz="0.044046 -0.007397 -0.050167" rpy="0 0 0"/>
     <geometry>
       <mesh filename="file://$(find bd1_bot_description)/meshes/right_bottom_leg_part1_1.stl" scale="0.001 0.001 0.001"/>
@@ -166,10 +166,10 @@
 <link name="right_bottom_leg_part2_1">
   <inertial>
-    <origin xyz="0.002889194540569691 0.030810626413684525 0.04744453662571095" rpy="0 0 0"/>
-    <mass value="0.01039775817481047"/>
-    <inertia ixx="1.3e-05" iyy="9e-06" izz="4e-06" ixy="-0.0" iyz="-5e-06" ixz="-0.0"/>
-  </inertial>
-  <visual>
-    <origin xyz="0.036046 -0.038191 -0.070137" rpy="0 0 0"/>
+    <origin xyz="0.0028891945405694133 0.030811277914758392 0.04744465826520479" rpy="0 0 0"/>
+    <mass value="0.00798668381543413"/>
+    <inertia ixx="1e-05" iyy="7e-06" izz="3e-06" ixy="-0.0" iyz="-4e-06" ixz="-0.0"/>
+  </inertial>
+  <visual>
+    <origin xyz="0.036046 -0.007397 -0.050167" rpy="0 0 0"/>
     <geometry>
       <mesh filename="file://$(find bd1_bot_description)/meshes/right_bottom_leg_part2_1.stl" scale="0.001 0.001 0.001"/>
@@ -178,5 +178,5 @@
   </visual>
   <collision>
-    <origin xyz="0.036046 -0.038191 -0.070137" rpy="0 0 0"/>
+    <origin xyz="0.036046 -0.007397 -0.050167" rpy="0 0 0"/>
     <geometry>
       <mesh filename="file://$(find bd1_bot_description)/meshes/right_bottom_leg_part2_1.stl" scale="0.001 0.001 0.001"/>
@@ -186,10 +186,10 @@
 <link name="left_bottom_leg_part1_1">
   <inertial>
-    <origin xyz="0.002889194540569559 0.030810626413683845 0.04744453662571098" rpy="0 0 0"/>
-    <mass value="0.01039775817481047"/>
-    <inertia ixx="1.3e-05" iyy="9e-06" izz="4e-06" ixy="-0.0" iyz="-5e-06" ixz="-0.0"/>
-  </inertial>
-  <visual>
-    <origin xyz="-0.042454 -0.038191 -0.070137" rpy="0 0 0"/>
+    <origin xyz="0.002889194540569226 0.03081127791475769 0.04744465826520482" rpy="0 0 0"/>
+    <mass value="0.00798668381543413"/>
+    <inertia ixx="1e-05" iyy="7e-06" izz="3e-06" ixy="-0.0" iyz="-4e-06" ixz="-0.0"/>
+  </inertial>
+  <visual>
+    <origin xyz="-0.042454 -0.007397 -0.050167" rpy="0 0 0"/>
     <geometry>
       <mesh filename="file://$(find bd1_bot_description)/meshes/left_bottom_leg_part1_1.stl" scale="0.001 0.001 0.001"/>
@@ -198,5 +198,5 @@
   </visual>
   <collision>
-    <origin xyz="-0.042454 -0.038191 -0.070137" rpy="0 0 0"/>
+    <origin xyz="-0.042454 -0.007397 -0.050167" rpy="0 0 0"/>
     <geometry>
       <mesh filename="file://$(find bd1_bot_description)/meshes/left_bottom_leg_part1_1.stl" scale="0.001 0.001 0.001"/>
@@ -206,10 +206,10 @@
 <link name="left_bottom_leg_part2_1">
   <inertial>
-    <origin xyz="-0.0028882648793389296 0.030810626413683984 0.047444536625710965" rpy="0 0 0"/>
-    <mass value="0.01039775817481047"/>
-    <inertia ixx="1.3e-05" iyy="9e-06" izz="4e-06" ixy="0.0" iyz="-5e-06" ixz="0.0"/>
-  </inertial>
-  <visual>
-    <origin xyz="-0.034454 -0.038191 -0.070137" rpy="0 0 0"/>
+    <origin xyz="-0.002888264879339214 0.030811277914757802 0.047444658265204845" rpy="0 0 0"/>
+    <mass value="0.00798668381543413"/>
+    <inertia ixx="1e-05" iyy="7e-06" izz="3e-06" ixy="0.0" iyz="-4e-06" ixz="0.0"/>
+  </inertial>
+  <visual>
+    <origin xyz="-0.034454 -0.007397 -0.050167" rpy="0 0 0"/>
     <geometry>
       <mesh filename="file://$(find bd1_bot_description)/meshes/left_bottom_leg_part2_1.stl" scale="0.001 0.001 0.001"/>
@@ -218,5 +218,5 @@
   </visual>
   <collision>
-    <origin xyz="-0.034454 -0.038191 -0.070137" rpy="0 0 0"/>
+    <origin xyz="-0.034454 -0.007397 -0.050167" rpy="0 0 0"/>
     <geometry>
       <mesh filename="file://$(find bd1_bot_description)/meshes/left_bottom_leg_part2_1.stl" scale="0.001 0.001 0.001"/>
@@ -226,10 +226,10 @@
 <link name="left_motor_1">
   <inertial>
-    <origin xyz="0.015112405129122444 1.3798701027981086e-07 -1.5177490494955315e-07" rpy="0 0 0"/>
-    <mass value="0.1704942333103181"/>
-    <inertia ixx="1.9e-05" iyy="2.3e-05" izz="2.3e-05" ixy="-0.0" iyz="0.0" ixz="0.0"/>
-  </inertial>
-  <visual>
-    <origin xyz="-0.029454 -0.030021 -0.057557" rpy="0 0 0"/>
+    <origin xyz="0.015112405129122132 -2.105119158497164e-07 -3.0135411110965293e-08" rpy="0 0 0"/>
+    <mass value="0.05754180374223235"/>
+    <inertia ixx="6e-06" iyy="8e-06" izz="8e-06" ixy="-0.0" iyz="0.0" ixz="0.0"/>
+  </inertial>
+  <visual>
+    <origin xyz="-0.029454 0.000772 -0.037587" rpy="0 0 0"/>
     <geometry>
       <mesh filename="file://$(find bd1_bot_description)/meshes/left_motor_1.stl" scale="0.001 0.001 0.001"/>
@@ -238,5 +238,5 @@
   </visual>
   <collision>
-    <origin xyz="-0.029454 -0.030021 -0.057557" rpy="0 0 0"/>
+    <origin xyz="-0.029454 0.000772 -0.037587" rpy="0 0 0"/>
     <geometry>
       <mesh filename="file://$(find bd1_bot_description)/meshes/left_motor_1.stl" scale="0.001 0.001 0.001"/>
@@ -246,10 +246,10 @@
 <link name="right_motor_1">
   <inertial>
-    <origin xyz="-0.015111475467892387 1.3798700971776046e-07 -1.5177490413770256e-07" rpy="0 0 0"/>
-    <mass value="0.1704942333103181"/>
-    <inertia ixx="1.9e-05" iyy="2.3e-05" izz="2.3e-05" ixy="-0.0" iyz="0.0" ixz="0.0"/>
-  </inertial>
-  <visual>
-    <origin xyz="0.031046 -0.030021 -0.057557" rpy="0 0 0"/>
+    <origin xyz="-0.015111475467892679 -2.10511916381626e-07 -3.013541029217581e-08" rpy="0 0 0"/>
+    <mass value="0.05754180374223235"/>
+    <inertia ixx="6e-06" iyy="8e-06" izz="8e-06" ixy="-0.0" iyz="0.0" ixz="0.0"/>
+  </inertial>
+  <visual>
+    <origin xyz="0.031046 0.000772 -0.037587" rpy="0 0 0"/>
     <geometry>
       <mesh filename="file://$(find bd1_bot_description)/meshes/right_motor_1.stl" scale="0.001 0.001 0.001"/>
@@ -258,5 +258,5 @@
   </visual>
   <collision>
-    <origin xyz="0.031046 -0.030021 -0.057557" rpy="0 0 0"/>
+    <origin xyz="0.031046 0.000772 -0.037587" rpy="0 0 0"/>
     <geometry>
       <mesh filename="file://$(find bd1_bot_description)/meshes/right_motor_1.stl" scale="0.001 0.001 0.001"/>
@@ -266,10 +266,10 @@
 <link name="left_wheel_1">
   <inertial>
-    <origin xyz="-0.004999534893301766 1.329023638918514e-07 -1.5890564092346793e-07" rpy="0 0 0"/>
-    <mass value="0.04003018480536562"/>
-    <inertia ixx="2.8e-05" iyy="1.5e-05" izz="1.5e-05" ixy="-0.0" iyz="-0.0" ixz="-0.0"/>
-  </inertial>
-  <visual>
-    <origin xyz="-0.074454 -0.030021 -0.057557" rpy="0 0 0"/>
+    <origin xyz="-0.004999534893302071 -2.1559656221566657e-07 -3.7266147084880075e-08" rpy="0 0 0"/>
+    <mass value="0.02988168724907574"/>
+    <inertia ixx="2.1e-05" iyy="1.1e-05" izz="1.1e-05" ixy="-0.0" iyz="-0.0" ixz="-0.0"/>
+  </inertial>
+  <visual>
+    <origin xyz="-0.074454 0.000772 -0.037587" rpy="0 0 0"/>
     <geometry>
       <mesh filename="file://$(find bd1_bot_description)/meshes/left_wheel_1.stl" scale="0.001 0.001 0.001"/>
@@ -278,5 +278,5 @@
   </visual>
   <collision>
-    <origin xyz="-0.074454 -0.030021 -0.057557" rpy="0 0 0"/>
+    <origin xyz="-0.074454 0.000772 -0.037587" rpy="0 0 0"/>
     <geometry>
       <mesh filename="file://$(find bd1_bot_description)/meshes/left_wheel_1.stl" scale="0.001 0.001 0.001"/>
@@ -286,10 +286,10 @@
 <link name="right_wheel_1">
   <inertial>
-    <origin xyz="0.005000464554531833 1.3354087039299523e-07 -1.593202911612246e-07" rpy="0 0 0"/>
-    <mass value="0.04003018480536562"/>
-    <inertia ixx="2.8e-05" iyy="1.5e-05" izz="1.5e-05" ixy="0.0" iyz="0.0" ixz="0.0"/>
-  </inertial>
-  <visual>
-    <origin xyz="0.076046 -0.030021 -0.057557" rpy="0 0 0"/>
+    <origin xyz="0.005000464554531528 -2.1495805572634055e-07 -3.7680797315697845e-08" rpy="0 0 0"/>
+    <mass value="0.02988168724907574"/>
+    <inertia ixx="2.1e-05" iyy="1.1e-05" izz="1.1e-05" ixy="0.0" iyz="0.0" ixz="0.0"/>
+  </inertial>
+  <visual>
+    <origin xyz="0.076046 0.000772 -0.037587" rpy="0 0 0"/>
     <geometry>
       <mesh filename="file://$(find bd1_bot_description)/meshes/right_wheel_1.stl" scale="0.001 0.001 0.001"/>
@@ -298,5 +298,5 @@
   </visual>
   <collision>
-    <origin xyz="0.076046 -0.030021 -0.057557" rpy="0 0 0"/>
+    <origin xyz="0.076046 0.000772 -0.037587" rpy="0 0 0"/>
     <geometry>
       <mesh filename="file://$(find bd1_bot_description)/meshes/right_wheel_1.stl" scale="0.001 0.001 0.001"/>
@@ -306,10 +306,10 @@
 <link name="left_tyre_1">
   <inertial>
-    <origin xyz="0.010019081554393537 1.3838490093773248e-07 -1.512219713339924e-07" rpy="0 0 0"/>
+    <origin xyz="0.010019081554393218 -2.101140251726044e-07 -2.958247750234344e-08" rpy="0 0 0"/>
     <mass value="0.024104122361266803"/>
     <inertia ixx="2.9e-05" iyy="1.6e-05" izz="1.6e-05" ixy="-0.0" iyz="-0.0" ixz="-0.0"/>
   </inertial>
   <visual>
-    <origin xyz="-0.059454 -0.030021 -0.057557" rpy="0 0 0"/>
+    <origin xyz="-0.059454 0.000772 -0.037587" rpy="0 0 0"/>
     <geometry>
       <mesh filename="file://$(find bd1_bot_description)/meshes/left_tyre_1.stl" scale="0.001 0.001 0.001"/>
@@ -318,5 +318,5 @@
   </visual>
   <collision>
-    <origin xyz="-0.059454 -0.030021 -0.057557" rpy="0 0 0"/>
+    <origin xyz="-0.059454 0.000772 -0.037587" rpy="0 0 0"/>
     <geometry>
       <mesh filename="file://$(find bd1_bot_description)/meshes/left_tyre_1.stl" scale="0.001 0.001 0.001"/>
@@ -326,10 +326,10 @@
 <link name="right_tyre_1">
   <inertial>
-    <origin xyz="-0.010018151893163477 1.3764371806571085e-07 -1.5236329475865062e-07" rpy="0 0 0"/>
+    <origin xyz="-0.010018151893163768 -2.1085520805666069e-07 -3.0723800906184984e-08" rpy="0 0 0"/>
     <mass value="0.024104122361266803"/>
     <inertia ixx="2.9e-05" iyy="1.6e-05" izz="1.6e-05" ixy="-0.0" iyz="-0.0" ixz="-0.0"/>
   </inertial>
   <visual>
-    <origin xyz="0.061046 -0.030021 -0.057557" rpy="0 0 0"/>
+    <origin xyz="0.061046 0.000772 -0.037587" rpy="0 0 0"/>
     <geometry>
       <mesh filename="file://$(find bd1_bot_description)/meshes/right_tyre_1.stl" scale="0.001 0.001 0.001"/>
@@ -338,5 +338,5 @@
   </visual>
   <collision>
-    <origin xyz="0.061046 -0.030021 -0.057557" rpy="0 0 0"/>
+    <origin xyz="0.061046 0.000772 -0.037587" rpy="0 0 0"/>
     <geometry>
       <mesh filename="file://$(find bd1_bot_description)/meshes/right_tyre_1.stl" scale="0.001 0.001 0.001"/>
@@ -346,10 +346,10 @@
 <link name="head_connector_1">
   <inertial>
-    <origin xyz="4.648306150260742e-07 0.035355109235206815 0.035355811907157364" rpy="0 0 0"/>
-    <mass value="0.07490342887208488"/>
-    <inertia ixx="8.1e-05" iyy="4.3e-05" izz="4.3e-05" ixy="-0.0" iyz="-3.6e-05" ixz="-0.0"/>
-  </inertial>
-  <visual>
-    <origin xyz="0.000296 0.005507 -0.229595" rpy="0 0 0"/>
+    <origin xyz="4.6483061472184705e-07 0.035355760736280634 0.03535493354665112" rpy="0 0 0"/>
+    <mass value="0.055913827186204204"/>
+    <inertia ixx="6e-05" iyy="3.2e-05" izz="3.2e-05" ixy="-0.0" iyz="-2.7e-05" ixz="-0.0"/>
+  </inertial>
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