Commit message: Updated COM

File: bd1_bot_description/urdf/bd1_bot.xacro (robot description, xacro)
@@ -6,5 +6,5 @@
 <link name="base_link">
   <inertial>
-    <origin xyz="-0.00032734350998203383 -0.03347164637300757 0.1802949431054025" rpy="0 0 0"/>
+    <origin xyz="-3.180834059638465e-05 -0.02893757368740919 0.17717056516547702" rpy="0 0 0"/>
     <mass value="0.6871683490298791"/>
     <inertia ixx="0.001278" iyy="0.000754" izz="0.001226" ixy="0.0" iyz="9e-06" ixz="-0.0"/>
@@ -26,10 +26,10 @@
 <link name="left_top_leg_1">
   <inertial>
-    <origin xyz="0.008147102971613591 0.039567400396896726 -0.014401308916336203" rpy="0 0 0"/>
+    <origin xyz="0.008146638140998697 0.0395674730824959 -0.014401686856261642" rpy="0 0 0"/>
     <mass value="0.11765454158339926"/>
     <inertia ixx="0.000238" iyy="5.5e-05" izz="0.000189" ixy="-6e-06" iyz="5.6e-05" ixz="2e-06"/>
   </inertial>
   <visual>
-    <origin xyz="-0.043454 0.021589 -0.179961" rpy="0 0 0"/>
+    <origin xyz="-0.04375 0.017055 -0.176837" rpy="0 0 0"/>
     <geometry>
       <mesh filename="file://$(find bd1_bot_description)/meshes/left_top_leg_1.stl" scale="0.001 0.001 0.001"/>
@@ -38,5 +38,5 @@
   </visual>
   <collision>
-    <origin xyz="-0.043454 0.021589 -0.179961" rpy="0 0 0"/>
+    <origin xyz="-0.04375 0.017055 -0.176837" rpy="0 0 0"/>
     <geometry>
       <mesh filename="file://$(find bd1_bot_description)/meshes/left_top_leg_1.stl" scale="0.001 0.001 0.001"/>
@@ -46,10 +46,10 @@
 <link name="right_top_leg_1">
   <inertial>
-    <origin xyz="-0.008146173310383774 0.03956740039699889 -0.014401308916058286" rpy="0 0 0"/>
+    <origin xyz="-0.008146638140998898 0.03956747308259668 -0.01440168685598367" rpy="0 0 0"/>
     <mass value="0.11765454158339926"/>
     <inertia ixx="0.000238" iyy="5.5e-05" izz="0.000189" ixy="6e-06" iyz="5.6e-05" ixz="-2e-06"/>
   </inertial>
   <visual>
-    <origin xyz="0.044046 0.021589 -0.179961" rpy="0 0 0"/>
+    <origin xyz="0.04375 0.017055 -0.176837" rpy="0 0 0"/>
     <geometry>
       <mesh filename="file://$(find bd1_bot_description)/meshes/right_top_leg_1.stl" scale="0.001 0.001 0.001"/>
@@ -58,5 +58,5 @@
   </visual>
   <collision>
-    <origin xyz="0.044046 0.021589 -0.179961" rpy="0 0 0"/>
+    <origin xyz="0.04375 0.017055 -0.176837" rpy="0 0 0"/>
     <geometry>
       <mesh filename="file://$(find bd1_bot_description)/meshes/right_top_leg_1.stl" scale="0.001 0.001 0.001"/>
@@ -66,10 +66,10 @@
 <link name="left_top_leg_part_1">
   <inertial>
-    <origin xyz="0.003017147690062824 -0.007158965723654645 0.002605836912960652" rpy="0 0 0"/>
+    <origin xyz="0.0030166828594480125 0.022791614835476554 -0.008295935118418557" rpy="0 0 0"/>
     <mass value="0.00355238590700276"/>
     <inertia ixx="1e-06" iyy="0.0" izz="1e-06" ixy="0.0" iyz="0.0" ixz="-0.0"/>
   </inertial>
   <visual>
-    <origin xyz="-0.057454 -0.019109 -0.165148" rpy="0 0 0"/>
+    <origin xyz="-0.05775 0.005408 -0.172598" rpy="0 0 0"/>
     <geometry>
       <mesh filename="file://$(find bd1_bot_description)/meshes/left_top_leg_part_1.stl" scale="0.001 0.001 0.001"/>
@@ -78,5 +78,5 @@
   </visual>
   <collision>
-    <origin xyz="-0.057454 -0.019109 -0.165148" rpy="0 0 0"/>
+    <origin xyz="-0.05775 0.005408 -0.172598" rpy="0 0 0"/>
     <geometry>
       <mesh filename="file://$(find bd1_bot_description)/meshes/left_top_leg_part_1.stl" scale="0.001 0.001 0.001"/>
@@ -86,10 +86,10 @@
 <link name="right_top_leg_part_1">
   <inertial>
-    <origin xyz="-0.0030162180288331314 -0.007158965723653446 0.002605836912960652" rpy="0 0 0"/>
+    <origin xyz="-0.0030166828594481512 0.022791614835476138 -0.008295935118418613" rpy="0 0 0"/>
     <mass value="0.00355238590700276"/>
     <inertia ixx="1e-06" iyy="0.0" izz="1e-06" ixy="-0.0" iyz="0.0" ixz="0.0"/>
   </inertial>
   <visual>
-    <origin xyz="0.058046 -0.019109 -0.165148" rpy="0 0 0"/>
+    <origin xyz="0.05775 0.005408 -0.172598" rpy="0 0 0"/>
     <geometry>
       <mesh filename="file://$(find bd1_bot_description)/meshes/right_top_leg_part_1.stl" scale="0.001 0.001 0.001"/>
@@ -98,5 +98,5 @@
   </visual>
   <collision>
-    <origin xyz="0.058046 -0.019109 -0.165148" rpy="0 0 0"/>
+    <origin xyz="0.05775 0.005408 -0.172598" rpy="0 0 0"/>
     <geometry>
       <mesh filename="file://$(find bd1_bot_description)/meshes/right_top_leg_part_1.stl" scale="0.001 0.001 0.001"/>
@@ -106,10 +106,10 @@
 <link name="left_bottom_leg_1">
   <inertial>
-    <origin xyz="-0.004999535169384971 -0.03183047151744199 -0.046387693982860134" rpy="0 0 0"/>
+    <origin xyz="-0.005000000000000122 -0.03342992083960998 -0.04524895101460043" rpy="0 0 0"/>
     <mass value="0.06694057104242657"/>
-    <inertia ixx="0.000154" iyy="0.0001" izz="5.5e-05" ixy="-0.0" iyz="-5.9e-05" ixz="-0.0"/>
-  </inertial>
-  <visual>
-    <origin xyz="-0.043454 -0.070031 -0.146614" rpy="0 0 0"/>
+    <inertia ixx="0.000154" iyy="9.6e-05" izz="5.9e-05" ixy="0.0" iyz="-6e-05" ixz="0.0"/>
+  </inertial>
+  <visual>
+    <origin xyz="-0.04375 -0.074565 -0.14349" rpy="0 0 0"/>
     <geometry>
       <mesh filename="file://$(find bd1_bot_description)/meshes/left_bottom_leg_1.stl" scale="0.001 0.001 0.001"/>
@@ -118,5 +118,5 @@
   </visual>
   <collision>
-    <origin xyz="-0.043454 -0.070031 -0.146614" rpy="0 0 0"/>
+    <origin xyz="-0.04375 -0.074565 -0.14349" rpy="0 0 0"/>
     <geometry>
       <mesh filename="file://$(find bd1_bot_description)/meshes/left_bottom_leg_1.stl" scale="0.001 0.001 0.001"/>
@@ -124,12 +124,52 @@
   </collision>
 </link>
+<link name="left_bottom_leg_part1_1">
+  <inertial>
+    <origin xyz="0.0028887297099540535 0.030804854644567246 0.043994677208628444" rpy="0 0 0"/>
+    <mass value="0.007986683815434131"/>
+    <inertia ixx="8e-06" iyy="6e-06" izz="3e-06" ixy="-0.0" iyz="-4e-06" ixz="-0.0"/>
+  </inertial>
+  <visual>
+    <origin xyz="-0.04275 -0.008604 -0.049287" rpy="0 0 0"/>
+    <geometry>
+      <mesh filename="file://$(find bd1_bot_description)/meshes/left_bottom_leg_part1_1.stl" scale="0.001 0.001 0.001"/>
+    </geometry>
+    <material name="silver"/>
+  </visual>
+  <collision>
+    <origin xyz="-0.04275 -0.008604 -0.049287" rpy="0 0 0"/>
+    <geometry>
+      <mesh filename="file://$(find bd1_bot_description)/meshes/left_bottom_leg_part1_1.stl" scale="0.001 0.001 0.001"/>
+    </geometry>
+  </collision>
+</link>
+<link name="left_bottom_leg_part2_1">
+  <inertial>
+    <origin xyz="-0.0028887297099543657 0.03080485464456717 0.043994677208628416" rpy="0 0 0"/>
+    <mass value="0.007986683815434131"/>
+    <inertia ixx="8e-06" iyy="6e-06" izz="3e-06" ixy="0.0" iyz="-4e-06" ixz="0.0"/>
+  </inertial>
+  <visual>
+    <origin xyz="-0.03475 -0.008604 -0.049287" rpy="0 0 0"/>
+    <geometry>
+      <mesh filename="file://$(find bd1_bot_description)/meshes/left_bottom_leg_part2_1.stl" scale="0.001 0.001 0.001"/>
+    </geometry>
+    <material name="silver"/>
+  </visual>
+  <collision>
+    <origin xyz="-0.03475 -0.008604 -0.049287" rpy="0 0 0"/>
+    <geometry>
+      <mesh filename="file://$(find bd1_bot_description)/meshes/left_bottom_leg_part2_1.stl" scale="0.001 0.001 0.001"/>
+    </geometry>
+  </collision>
+</link>
 <link name="right_bottom_leg_1">
   <inertial>
-    <origin xyz="0.004000464830615148 -0.03183047151744129 -0.04638769398286016" rpy="0 0 0"/>
+    <origin xyz="0.004999999999999803 -0.03342992083961032 -0.045248951014600344" rpy="0 0 0"/>
     <mass value="0.06694057104242657"/>
-    <inertia ixx="0.000154" iyy="0.0001" izz="5.5e-05" ixy="-0.0" iyz="-5.9e-05" ixz="-0.0"/>
-  </inertial>
-  <visual>
-    <origin xyz="0.044046 -0.070031 -0.146614" rpy="0 0 0"/>
+    <inertia ixx="0.000154" iyy="9.6e-05" izz="5.9e-05" ixy="0.0" iyz="-6e-05" ixz="0.0"/>
+  </inertial>
+  <visual>
+    <origin xyz="0.04375 -0.074565 -0.14349" rpy="0 0 0"/>
     <geometry>
       <mesh filename="file://$(find bd1_bot_description)/meshes/right_bottom_leg_1.stl" scale="0.001 0.001 0.001"/>
@@ -138,5 +178,5 @@
   </visual>
   <collision>
-    <origin xyz="0.044046 -0.070031 -0.146614" rpy="0 0 0"/>
+    <origin xyz="0.04375 -0.074565 -0.14349" rpy="0 0 0"/>
     <geometry>
       <mesh filename="file://$(find bd1_bot_description)/meshes/right_bottom_leg_1.stl" scale="0.001 0.001 0.001"/>
@@ -146,10 +186,10 @@
 <link name="right_bottom_leg_part1_1">
   <inertial>
-    <origin xyz="-0.002888264879339103 0.030811277914758503 0.04744465826520482" rpy="0 0 0"/>
-    <mass value="0.00798668381543413"/>
-    <inertia ixx="1e-05" iyy="7e-06" izz="3e-06" ixy="0.0" iyz="-4e-06" ixz="0.0"/>
-  </inertial>
-  <visual>
-    <origin xyz="0.044046 -0.007397 -0.050167" rpy="0 0 0"/>
+    <origin xyz="-0.0028887297099544212 0.03080485464456685 0.0439946772086285" rpy="0 0 0"/>
+    <mass value="0.007986683815434131"/>
+    <inertia ixx="8e-06" iyy="6e-06" izz="3e-06" ixy="0.0" iyz="-4e-06" ixz="0.0"/>
+  </inertial>
+  <visual>
+    <origin xyz="0.04275 -0.008604 -0.049287" rpy="0 0 0"/>
     <geometry>
       <mesh filename="file://$(find bd1_bot_description)/meshes/right_bottom_leg_part1_1.stl" scale="0.001 0.001 0.001"/>
@@ -158,5 +198,5 @@
   </visual>
   <collision>
-    <origin xyz="0.044046 -0.007397 -0.050167" rpy="0 0 0"/>
+    <origin xyz="0.04275 -0.008604 -0.049287" rpy="0 0 0"/>
     <geometry>
       <mesh filename="file://$(find bd1_bot_description)/meshes/right_bottom_leg_part1_1.stl" scale="0.001 0.001 0.001"/>
@@ -166,10 +206,10 @@
 <link name="right_bottom_leg_part2_1">
   <inertial>
-    <origin xyz="0.0028891945405694133 0.030811277914758392 0.04744465826520479" rpy="0 0 0"/>
-    <mass value="0.00798668381543413"/>
-    <inertia ixx="1e-05" iyy="7e-06" izz="3e-06" ixy="-0.0" iyz="-4e-06" ixz="-0.0"/>
-  </inertial>
-  <visual>
-    <origin xyz="0.036046 -0.007397 -0.050167" rpy="0 0 0"/>
+    <origin xyz="0.002888729709954102 0.03080485464456688 0.04399467720862853" rpy="0 0 0"/>
+    <mass value="0.007986683815434131"/>
+    <inertia ixx="8e-06" iyy="6e-06" izz="3e-06" ixy="-0.0" iyz="-4e-06" ixz="-0.0"/>
+  </inertial>
+  <visual>
+    <origin xyz="0.03475 -0.008604 -0.049287" rpy="0 0 0"/>
     <geometry>
       <mesh filename="file://$(find bd1_bot_description)/meshes/right_bottom_leg_part2_1.stl" scale="0.001 0.001 0.001"/>
@@ -178,5 +218,5 @@
   </visual>
   <collision>
-    <origin xyz="0.036046 -0.007397 -0.050167" rpy="0 0 0"/>
+    <origin xyz="0.03475 -0.008604 -0.049287" rpy="0 0 0"/>
     <geometry>
       <mesh filename="file://$(find bd1_bot_description)/meshes/right_bottom_leg_part2_1.stl" scale="0.001 0.001 0.001"/>
@@ -184,52 +224,12 @@
   </collision>
 </link>
-<link name="left_bottom_leg_part1_1">
-  <inertial>
-    <origin xyz="0.002889194540569226 0.03081127791475769 0.04744465826520482" rpy="0 0 0"/>
-    <mass value="0.00798668381543413"/>
-    <inertia ixx="1e-05" iyy="7e-06" izz="3e-06" ixy="-0.0" iyz="-4e-06" ixz="-0.0"/>
-  </inertial>
-  <visual>
-    <origin xyz="-0.042454 -0.007397 -0.050167" rpy="0 0 0"/>
-    <geometry>
-      <mesh filename="file://$(find bd1_bot_description)/meshes/left_bottom_leg_part1_1.stl" scale="0.001 0.001 0.001"/>
-    </geometry>
-    <material name="silver"/>
-  </visual>
-  <collision>
-    <origin xyz="-0.042454 -0.007397 -0.050167" rpy="0 0 0"/>
-    <geometry>
-      <mesh filename="file://$(find bd1_bot_description)/meshes/left_bottom_leg_part1_1.stl" scale="0.001 0.001 0.001"/>
-    </geometry>
-  </collision>
-</link>
-<link name="left_bottom_leg_part2_1">
-  <inertial>
-    <origin xyz="-0.002888264879339214 0.030811277914757802 0.047444658265204845" rpy="0 0 0"/>
-    <mass value="0.00798668381543413"/>
-    <inertia ixx="1e-05" iyy="7e-06" izz="3e-06" ixy="0.0" iyz="-4e-06" ixz="0.0"/>
-  </inertial>
-  <visual>
-    <origin xyz="-0.034454 -0.007397 -0.050167" rpy="0 0 0"/>
-    <geometry>
-      <mesh filename="file://$(find bd1_bot_description)/meshes/left_bottom_leg_part2_1.stl" scale="0.001 0.001 0.001"/>
-    </geometry>
-    <material name="silver"/>
-  </visual>
-  <collision>
-    <origin xyz="-0.034454 -0.007397 -0.050167" rpy="0 0 0"/>
-    <geometry>
-      <mesh filename="file://$(find bd1_bot_description)/meshes/left_bottom_leg_part2_1.stl" scale="0.001 0.001 0.001"/>
-    </geometry>
-  </collision>
-</link>
 <link name="left_motor_1">
   <inertial>
-    <origin xyz="0.015112405129122132 -2.105119158497164e-07 -3.0135411110965293e-08" rpy="0 0 0"/>
-    <mass value="0.05754180374223235"/>
-    <inertia ixx="6e-06" iyy="8e-06" izz="8e-06" ixy="-0.0" iyz="0.0" ixz="0.0"/>
-  </inertial>
-  <visual>
-    <origin xyz="-0.029454 0.000772 -0.037587" rpy="0 0 0"/>
+    <origin xyz="0.015111940298507473 7.507795174563197e-16 -4.996003610813204e-16" rpy="0 0 0"/>
+    <mass value="0.022590485913617148"/>
+    <inertia ixx="3e-06" iyy="3e-06" izz="3e-06" ixy="-0.0" iyz="0.0" ixz="0.0"/>
+  </inertial>
+  <visual>
+    <origin xyz="-0.02975 -0.0 -0.037" rpy="0 0 0"/>
     <geometry>
       <mesh filename="file://$(find bd1_bot_description)/meshes/left_motor_1.stl" scale="0.001 0.001 0.001"/>
@@ -238,5 +238,5 @@
   </visual>
   <collision>
-    <origin xyz="-0.029454 0.000772 -0.037587" rpy="0 0 0"/>
+    <origin xyz="-0.02975 -0.0 -0.037" rpy="0 0 0"/>
     <geometry>
       <mesh filename="file://$(find bd1_bot_description)/meshes/left_motor_1.stl" scale="0.001 0.001 0.001"/>
@@ -244,12 +244,52 @@
   </collision>
 </link>
+<link name="left_wheel_1">
+  <inertial>
+    <origin xyz="-0.004999999723916709 5.330407374826963e-09 6.948940922679725e-09" rpy="0 0 0"/>
+    <mass value="0.02988168724907574"/>
+    <inertia ixx="2.1e-05" iyy="1.1e-05" izz="1.1e-05" ixy="0.0" iyz="-0.0" ixz="0.0"/>
+  </inertial>
+  <visual>
+    <origin xyz="-0.07475 -0.0 -0.037" rpy="0 0 0"/>
+    <geometry>
+      <mesh filename="file://$(find bd1_bot_description)/meshes/left_wheel_1.stl" scale="0.001 0.001 0.001"/>
+    </geometry>
+    <material name="silver"/>
+  </visual>
+  <collision>
+    <origin xyz="-0.07475 -0.0 -0.037" rpy="0 0 0"/>
+    <geometry>
+      <mesh filename="file://$(find bd1_bot_description)/meshes/left_wheel_1.stl" scale="0.001 0.001 0.001"/>
+    </geometry>
+  </collision>
+</link>
+<link name="left_tyre_1">
+  <inertial>
+    <origin xyz="-1.858665114175262e-05 3.4965965086175387e-10 5.557722476678961e-10" rpy="0 0 0"/>
+    <mass value="0.027473313011808588"/>
+    <inertia ixx="3.3e-05" iyy="1.8e-05" izz="1.8e-05" ixy="0.0" iyz="-0.0" ixz="0.0"/>
+  </inertial>
+  <visual>
+    <origin xyz="-0.06975 -0.0 -0.037" rpy="0 0 0"/>
+    <geometry>
+      <mesh filename="file://$(find bd1_bot_description)/meshes/left_tyre_1.stl" scale="0.001 0.001 0.001"/>
+    </geometry>
+    <material name="silver"/>
+  </visual>
+  <collision>
+    <origin xyz="-0.06975 -0.0 -0.037" rpy="0 0 0"/>
+    <geometry>
+      <mesh filename="file://$(find bd1_bot_description)/meshes/left_tyre_1.stl" scale="0.001 0.001 0.001"/>
+    </geometry>
+  </collision>
+</link>
 <link name="right_motor_1">
   <inertial>
-    <origin xyz="-0.015111475467892679 -2.10511916381626e-07 -3.013541029217581e-08" rpy="0 0 0"/>
-    <mass value="0.05754180374223235"/>
-    <inertia ixx="6e-06" iyy="8e-06" izz="8e-06" ixy="-0.0" iyz="0.0" ixz="0.0"/>
-  </inertial>
-  <visual>
-    <origin xyz="0.031046 0.000772 -0.037587" rpy="0 0 0"/>
+    <origin xyz="-0.015111940298507438 -9.605255930854404e-16 5.065392549852277e-16" rpy="0 0 0"/>
+    <mass value="0.022590485913617148"/>
+    <inertia ixx="3e-06" iyy="3e-06" izz="3e-06" ixy="-0.0" iyz="0.0" ixz="0.0"/>
+  </inertial>
+  <visual>
+    <origin xyz="0.02975 0.0 -0.037" rpy="0 0 0"/>
     <geometry>
       <mesh filename="file://$(find bd1_bot_description)/meshes/right_motor_1.stl" scale="0.001 0.001 0.001"/>
@@ -258,5 +298,5 @@
   </visual>
   <collision>
-    <origin xyz="0.031046 0.000772 -0.037587" rpy="0 0 0"/>
+    <origin xyz="0.02975 0.0 -0.037" rpy="0 0 0"/>
     <geometry>
       <mesh filename="file://$(find bd1_bot_description)/meshes/right_motor_1.stl" scale="0.001 0.001 0.001"/>
@@ -264,32 +304,12 @@
   </collision>
 </link>
-<link name="left_wheel_1">
-  <inertial>
-    <origin xyz="-0.004999534893302071 -2.1559656221566657e-07 -3.7266147084880075e-08" rpy="0 0 0"/>
+<link name="right_wheel_1">
+  <inertial>
+    <origin xyz="0.00500000042509488 5.330406753102071e-09 6.94894101982424e-09" rpy="0 0 0"/>
     <mass value="0.02988168724907574"/>
-    <inertia ixx="2.1e-05" iyy="1.1e-05" izz="1.1e-05" ixy="-0.0" iyz="-0.0" ixz="-0.0"/>
-  </inertial>
-  <visual>
-    <origin xyz="-0.074454 0.000772 -0.037587" rpy="0 0 0"/>
-    <geometry>
-      <mesh filename="file://$(find bd1_bot_description)/meshes/left_wheel_1.stl" scale="0.001 0.001 0.001"/>
-    </geometry>
-    <material name="silver"/>
-  </visual>
-  <collision>
-    <origin xyz="-0.074454 0.000772 -0.037587" rpy="0 0 0"/>
-    <geometry>
-      <mesh filename="file://$(find bd1_bot_description)/meshes/left_wheel_1.stl" scale="0.001 0.001 0.001"/>
-    </geometry>
-  </collision>
-</link>
-<link name="right_wheel_1">
-  <inertial>
-    <origin xyz="0.005000464554531528 -2.1495805572634055e-07 -3.7680797315697845e-08" rpy="0 0 0"/>
-    <mass value="0.02988168724907574"/>
-    <inertia ixx="2.1e-05" iyy="1.1e-05" izz="1.1e-05" ixy="0.0" iyz="0.0" ixz="0.0"/>
-  </inertial>
-  <visual>
-    <origin xyz="0.076046 0.000772 -0.037587" rpy="0 0 0"/>
+    <inertia ixx="2.1e-05" iyy="1.1e-05" izz="1.1e-05" ixy="0.0" iyz="-0.0" ixz="0.0"/>
+  </inertial>
+  <visual>
+    <origin xyz="0.07475 0.0 -0.037" rpy="0 0 0"/>
     <geometry>
       <mesh filename="file://$(find bd1_bot_description)/meshes/right_wheel_1.stl" scale="0.001 0.001 0.001"/>
@@ -298,5 +318,5 @@
   </visual>
   <collision>
-    <origin xyz="0.076046 0.000772 -0.037587" rpy="0 0 0"/>
+    <origin xyz="0.07475 0.0 -0.037" rpy="0 0 0"/>
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
Commit message: Updated Bot Design

File: bd1_bot_description/urdf/bd1_bot.xacro (robot description, xacro)
@@ -6,5 +6,5 @@
 <link name="base_link">
   <inertial>
-    <origin xyz="-3.180834059638465e-05 -0.02893757368740919 0.17717056516547702" rpy="0 0 0"/>
+    <origin xyz="-3.180834059638465e-05 -0.028937573687409172 0.17717056516547702" rpy="0 0 0"/>
     <mass value="0.6871683490298791"/>
     <inertia ixx="0.001278" iyy="0.000754" izz="0.001226" ixy="0.0" iyz="9e-06" ixz="-0.0"/>
@@ -26,7 +26,7 @@
 <link name="left_top_leg_1">
   <inertial>
-    <origin xyz="0.008146638140998697 0.0395674730824959 -0.014401686856261642" rpy="0 0 0"/>
-    <mass value="0.11765454158339926"/>
-    <inertia ixx="0.000238" iyy="5.5e-05" izz="0.000189" ixy="-6e-06" iyz="5.6e-05" ixz="2e-06"/>
+    <origin xyz="0.008170600100975256 0.0394894379137513 -0.014373284377612094" rpy="0 0 0"/>
+    <mass value="0.11806434962739475"/>
+    <inertia ixx="0.000239" iyy="5.5e-05" izz="0.00019" ixy="-6e-06" iyz="5.6e-05" ixz="2e-06"/>
   </inertial>
   <visual>
@@ -366,7 +366,7 @@
 <link name="head_1">
   <inertial>
-    <origin xyz="-1.9567650462359864e-06 -0.02143844644089888 0.008932494875529162" rpy="0 0 0"/>
-    <mass value="1.1993912366195452"/>
-    <inertia ixx="0.003148" iyy="0.002464" izz="0.005147" ixy="0.0" iyz="4.1e-05" ixz="0.0"/>
+    <origin xyz="-1.7784182525826254e-06 -0.021451548337959786 0.00893485011990891" rpy="0 0 0"/>
+    <mass value="1.199572908129388"/>
+    <inertia ixx="0.00315" iyy="0.002464" izz="0.005149" ixy="0.0" iyz="4.1e-05" ixz="0.0"/>
   </inertial>
   <visual>

Commit message: removed fake inertia

File: bd1_bot_description/urdf/bd1_bot.xacro (robot description, xacro)
@@ -605,9 +605,5 @@
 </link>
 <link name="fake_camera_1">
-  <inertial>
-    <origin xyz="-0.00010062533325747048 -0.0056682682583362315 0.0002650247252930782" rpy="0 0 0"/>
-    <mass value="0.0056389881980399275"/>
-    <inertia ixx="1e-06" iyy="1e-06" izz="1e-06" ixy="0.0" iyz="-0.0" ixz="0.0"/>
-  </inertial>
+  <origin xyz="-0.00010062533325747048 -0.0056682682583362315 0.0002650247252930782" rpy="0 0 0"/>
 </link>
 <joint name="left_top_leg_fix" type="fixed">
